Commit message: created yaml file for gazebo controller manager

File: description/ros2_control.xacro (robot description, xacro)
@@ -2,4 +2,27 @@
 <robot xmlns:xacro="http://www.ros.org/wiki/xacro">
     <ros2_control name="GazeboSystem" type="system">
+        <hardware>
+            <!-- The plugin is our hardware interface -->
+            <plugin><gazebo_ros2_control/GazeboSystem/plugin>
+        </hardware>
+        <joint name="left_wheel_joint">
+            <command_interface name="velocity">
+                <param name="min">-10</param>
+                <param name="max">10</param>
+            </command_interface>
+            <state_interface name="velocity"/>
+            <state_interface name="position"/>
+        </joint>
+        <joint name="right_wheel_joint">
+            <command_interface name="velocity">
+                <param name="min">-10</param>
+                <param name="max">10</param>
+            </command_interface>
+            <state_interface name="velocity"/>
+            <state_interface name="position"/>
+        </joint>
+        <gazebo>
+            <plugin name="gazebo_ros2_control" filename="libgazebo_ros2_control.so"></plugin>
+        </gazebo>
     </ros2_control>
 </robot>
